File: Reflow_Touch_shield_ESP32/Reflow_Touch_shield_ESP32.kicad_pcb (KiCad board)
At the start: 2 copper layers, 88.5 x 52.5 mm, 35 parts, among them IC1 MAX6675, J1 Conn_01x14, J2 Jack-DC, J3 , Q1 FDN340P, U1 LM358, U2 AMS1117-3.3, U3 ESP32-WROOM-32D, U4 AMS1117-5.0, U5 CH340C

Commit message: update
Parts:
- removed C1, C3, C7, C8: 100nF, Capacitor_SMD:C_0603_1608Metric_Pad1.08x0.95mm_HandSolder
- removed C2, C4: 10uF, Capacitor_SMD:C_0603_1608Metric_Pad1.08x0.95mm_HandSolder
- removed C5, C6: 47uF, Capacitor_SMD:CP_Elec_4x3
- removed C9: 100nf, Capacitor_SMD:C_0603_1608Metric_Pad1.08x0.95mm_HandSolder
- removed D1, D3, D4, D5: LED, LED_SMD:LED_0603_1608Metric_Pad1.05x0.95mm_HandSolder
- removed D2: DIODE, Diode_SMD:D_SOD-128
- removed J2: Jack-DC, Connector_BarrelJack:BarrelJack_Horizontal
- removed J3: , kien242:USB-C-16pin-hight-v2
- removed Q1: FDN340P, Package_TO_SOT_SMD:SOT-23_Handsoldering
- removed R1, R2: 10k, Resistor_SMD:R_0603_1608Metric_Pad0.98x0.95mm_HandSolder
- removed R10, R11, R3, R4, R5, R6, R7: 1K, Resistor_SMD:R_0603_1608Metric_Pad0.98x0.95mm_HandSolder
- removed R8, R9: 5.1K, Resistor_SMD:R_0603_1608Metric_Pad0.98x0.95mm_HandSolder
- removed U1: LM358, Package_SO:SOP-8_3.9x4.9mm_P1.27mm
- removed U2: AMS1117-3.3, Package_TO_SOT_SMD:SOT-223-3_TabPin2
- removed U3: ESP32-WROOM-32D, RF_Module:ESP32-WROOM-32
- removed U4: AMS1117-5.0, Package_TO_SOT_SMD:SOT-223-3_TabPin2
- removed U5: CH340C, Package_SO:SOIC-16_3.9x9.9mm_P1.27mm
- added A1: Arduino_UNO_R3, Module:Arduino_UNO_R3, B.Cu at (139.1, 48.9)
Routing:
- net D+: track 21.7 -> 0.00 mm
- net D-: track 20.8 -> 0.00 mm
- net Net-(J3-PadA5): track 3.64 -> 0.00 mm
- net Net-(J3-PadB5): track 3.43 -> 0.00 mm

Commit message: Update PCB
Parts:
- A1: footprint Module:Arduino_UNO_R3 -> Module:Arduino_UNO_R3_WithMountingHoles
Other:
- board size 88.5 x 52.5 mm -> 88.5 x 53.8 mm

Commit message: Update PCB
Parts:
- added BZ1: Buzzer, Buzzer_Beeper:MagneticBuzzer_CUI_CMT-8504-100-SMT, B.Cu at (147.9, 59.5)
- added C1: 0.1uF, Capacitor_SMD:C_0603_1608Metric_Pad1.08x0.95mm_HandSolder, B.Cu at (153.0, 82.2)
- added D1: D, Diode_SMD:D_SOD-123, B.Cu at (153.5, 87.6)
- added D2: D, Diode_SMD:D_SOD-123, B.Cu at (153.5, 69.9)
- added J1: Conn_01x02, TerminalBlock_Phoenix:TerminalBlock_Phoenix_MKDS-1,5-2-5.08_1x02_P5.08mm_Horizontal, B.Cu at (162.9, 56.7)
- added J2: Temp, Connector_JST:JST_EH_S2B-EH_1x02_P2.50mm_Horizontal, B.Cu at (161.0, 80.0)
- added J4: SSR, Connector_JST:JST_EH_S2B-EH_1x02_P2.50mm_Horizontal, B.Cu at (161.0, 71.1)
- added J5: Fan, Connector_JST:JST_EH_S2B-EH_1x02_P2.50mm_Horizontal, B.Cu at (161.0, 88.9)
- added Q1: AO3400A, Package_TO_SOT_SMD:SOT-23_Handsoldering, B.Cu at (149.3, 69.8)
- added Q2: AO3400A, Package_TO_SOT_SMD:SOT-23_Handsoldering, B.Cu at (149.3, 87.6)
- added Q3: AO3400A, Package_TO_SOT_SMD:SOT-23_Handsoldering, B.Cu at (139.2, 63.1)
- added R1: R, Resistor_SMD:R_0603_1608Metric_Pad0.98x0.95mm_HandSolder, B.Cu at (145.6, 69.8)
- added R2: R, Resistor_SMD:R_0603_1608Metric_Pad0.98x0.95mm_HandSolder, B.Cu at (145.6, 87.6)
- added R3: R, Resistor_SMD:R_0603_1608Metric_Pad0.98x0.95mm_HandSolder, B.Cu at (135.7, 63.1)
- added kibuzzard-632DE383: G***, kibuzzard-632DE383, B.Cu at (156.2, 69.8)
- added kibuzzard-632DE399: G***, kibuzzard-632DE399, B.Cu at (156.2, 87.6)
- added kibuzzard-632DE3A2: G***, kibuzzard-632DE3A2, B.Cu at (156.2, 78.7)
- added kibuzzard-632DE3CE: G***, kibuzzard-632DE3CE, B.Cu at (156.2, 59.4)
- A1: footprint Module:Arduino_UNO_R3_WithMountingHoles -> Module:Arduino_UNO_R3
- moved IC1 19.7 mm to (149.4, 78.7), turned to -90 degrees
- moved A1 12.2 mm to (126.9, 48.9)
- renumbered J1 to J3
Connections:
- A1 pad 10: unconnected-(A1-Pad10) -> heater_pins
- A1 pad 11: unconnected-(A1-Pad11) -> FAN
- A1 pad 17: unconnected-(A1-Pad17) -> IRQ_TOUCH
- A1 pad 18: unconnected-(A1-Pad18) -> CS_TOUCH
- A1 pad 19: unconnected-(A1-Pad19) -> LED_DISPLAY
- A1 pad 20: unconnected-(A1-Pad20) -> DC_DISPLAY
- A1 pad 21: unconnected-(A1-Pad21) -> RST_DISPLAY
- A1 pad 22: unconnected-(A1-Pad22) -> CS_DISPLAY
- A1 pad 23: unconnected-(A1-Pad23) -> CS_MISO
- A1 pad 24: unconnected-(A1-Pad24) -> CS_TEMP
- A1 pad 25: unconnected-(A1-Pad25) -> CS_SCK
- A1 pad 26: unconnected-(A1-Pad26) -> MOSI
- A1 pad 27: unconnected-(A1-Pad27) -> MISO
- A1 pad 28: unconnected-(A1-Pad28) -> SCK
- A1 pad 29: unconnected-(A1-Pad29) -> GND
- A1 pad 4: unconnected-(A1-Pad4) -> +3.3V
- A1 pad 5: unconnected-(A1-Pad5) -> +5V
- A1 pad 6: unconnected-(A1-Pad6) -> GND
- A1 pad 7: unconnected-(A1-Pad7) -> GND
- A1 pad 8: unconnected-(A1-Pad8) -> V-IN
- A1 pad 9: unconnected-(A1-Pad9) -> BUZZER
- IC1 pad 2: T- -> Net-(IC1-Pad2)
- IC1 pad 3: T+ -> Net-(IC1-Pad3)
- IC1 pad 5: SCK_TEMP -> CS_SCK
- IC1 pad 7: DO_TEMP -> CS_MISO
Routing:
- net +3.3V: track 0.00 -> 106.1 mm, vias 0 -> 2
- net +5V: track 0.00 -> 99.3 mm
- net FAN: track 0.00 -> 93.7 mm
- net SCK: track 0.00 -> 69.6 mm
- net MOSI: track 0.00 -> 69.0 mm, vias 0 -> 1
- net heater_pins: track 0.00 -> 68.2 mm
- net MISO: track 0.00 -> 64.2 mm, vias 0 -> 1
- net V-IN: track 0.00 -> 61.8 mm
- net CS_DISPLAY: track 0.00 -> 61.7 mm
- net RST_DISPLAY: track 0.00 -> 56.6 mm
- net CS_MISO: track 0.00 -> 52.1 mm
- net DC_DISPLAY: track 0.00 -> 51.5 mm
- net BUZZER: track 0.00 -> 48.9 mm
- net CS_TEMP: track 0.00 -> 48.3 mm
- net CS_SCK: track 0.00 -> 44.5 mm
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- added copper zone on B.Cu, net (none)
- added copper zone on F.Cu, net (none)
Other:
- board text added: "+"
- board text added: "-"
- board text removed: "2.8{dblquote} TFT Screen with touch sensor"
