File: Reflow_Touch_shield_ESP32/Reflow_Touch_shield_ESP32.kicad_sch (KiCad schematic)
At the start: 38 parts, among them IC1 MAX6675, J1 Conn_01x14, J2 Jack-DC, J3 , J4 Conn_01x04_MountingPin, Q1 FDN340P, SW1 SW_Push, U1 LM358, U2 AMS1117-3.3, U3 ESP32-WROOM-32D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

Commit message: update
Parts:
- removed C1, C3, C7, C8: 100nF, Capacitor_SMD:C_0603_1608Metric_Pad1.08x0.95mm_HandSolder, symbol stormduino-Rev2-rescue:C-Device
- removed C2, C4: 10uF, Capacitor_SMD:C_0603_1608Metric_Pad1.08x0.95mm_HandSolder, symbol stormduino-Rev2-rescue:C-Device
- removed C5, C6: 47uF, Capacitor_SMD:CP_Elec_4x3, symbol stormduino-Rev2-rescue:CP-Device
- removed C9: 100nf, Capacitor_SMD:C_0603_1608Metric_Pad1.08x0.95mm_HandSolder, symbol stormduino-Rev2-rescue:C-Device
- removed D1, D3, D4, D5: LED, LED_SMD:LED_0603_1608Metric_Pad1.05x0.95mm_HandSolder, symbol stormduino-Rev2-rescue:LED-Device
- removed D2: DIODE, Diode_SMD:D_SOD-128, symbol stormduino-Rev2-rescue:DIODE-pspice
- removed F1: Fuse, symbol stormduino-Rev2-rescue:Fuse-Device
- removed J2: Jack-DC, Connector_BarrelJack:BarrelJack_Horizontal, symbol stormduino-Rev2-rescue:Jack-DC-Connector
- removed J3: (no value), kien242:USB-C-16pin-hight-v2, symbol Connector:USB_C_Receptacle_USB2.0
- removed J4: Conn_01x04_MountingPin, symbol stormduino-Rev2-rescue:Conn_01x04_MountingPin-Connector_Generic_MountingPin
- removed Q1: FDN340P, Package_TO_SOT_SMD:SOT-23_Handsoldering, symbol Transistor_FET:FDN340P
- removed R1, R2: 10k, Resistor_SMD:R_0603_1608Metric_Pad0.98x0.95mm_HandSolder, symbol stormduino-Rev2-rescue:R-Device
- removed R10, R11, R3, R4, R5, R6, R7: 1K, Resistor_SMD:R_0603_1608Metric_Pad0.98x0.95mm_HandSolder, symbol stormduino-Rev2-rescue:R-Device
- removed R8, R9: 5.1K, Resistor_SMD:R_0603_1608Metric_Pad0.98x0.95mm_HandSolder, symbol stormduino-Rev2-rescue:R-Device
- removed SW1: SW_Push, symbol stormduino-Rev2-rescue:SW_Push-Switch
- removed U1: LM358, Package_SO:SOP-8_3.9x4.9mm_P1.27mm, symbol stormduino-Rev2-rescue:LM358-Amplifier_Operational
- removed U2: AMS1117-3.3, Package_TO_SOT_SMD:SOT-223-3_TabPin2, symbol stormduino-Rev2-rescue:AMS1117-3.3-Regulator_Linear
- removed U3: ESP32-WROOM-32D, RF_Module:ESP32-WROOM-32, symbol RF_Module:ESP32-WROOM-32D
- removed U4: AMS1117-5.0, Package_TO_SOT_SMD:SOT-223-3_TabPin2, symbol stormduino-Rev2-rescue:AMS1117-5.0-Regulator_Linear
- removed U5: CH340C, Package_SO:SOIC-16_3.9x9.9mm_P1.27mm, symbol stormduino-Rev2-rescue:CH340G-Interface_USB
- added A?: Arduino_UNO_R3, Module:Arduino_UNO_R3, symbol MCU_Module:Arduino_UNO_R3
Connections:
- no-connect marks 5 -> 0
Other:
- note removed: "LEDS"
- note removed: "POWER SUPPLY"
- note removed: "RESET SWITCH"
- note removed: "UART BREAKOUT HEADER"
- note removed: "USB TO UART"
- moved on the sheet: J1

Commit message: Update PCB
Parts:
- A1: renamed from A?; footprint Module:Arduino_UNO_R3 -> Module:Arduino_UNO_R3_WithMountingHoles
Changed lines of the file:
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@@
   (symbol (lib_id "power:+3.3V") (at 110.49 107.95 90) (mirror x) (unit 1)
     (in_bom yes) (on_board yes) (fields_autoplaced)
-    (property "Reference" "#PWR013" (id 0) (at 114.3 107.95 0)
+    (property "Reference" "#PWR04" (id 0) (at 114.3 107.95 0)
       (effects (font (size 1.27 1.27)) hide)
     )
@@
   (symbol (lib_id "power:GND") (at 110.49 105.41 270) (mirror x) (unit 1)
     (in_bom yes) (on_board yes) (fields_autoplaced)
-    (property "Reference" "#PWR012" (id 0) (at 104.14 105.41 0)
+    (property "Reference" "#PWR03" (id 0) (at 104.14 105.41 0)
       (effects (font (size 1.27 1.27)) hide)
     )
@@
   (symbol (lib_id "power:GND") (at 142.24 33.655 270) (unit 1)
     (in_bom yes) (on_board yes) (fields_autoplaced)
-    (property "Reference" "#PWR04" (id 0) (at 135.89 33.655 0)
+    (property "Reference" "#PWR01" (id 0) (at 135.89 33.655 0)
       (effects (font (size 1.27 1.27)) hide)
     )
@@
   (symbol (lib_id "power:+3.3V") (at 142.24 46.355 90) (unit 1)
     (in_bom yes) (on_board yes) (fields_autoplaced)
-    (property "Reference" "#PWR07" (id 0) (at 146.05 46.355 0)
+    (property "Reference" "#PWR02" (id 0) (at 146.05 46.355 0)
       (effects (font (size 1.27 1.27)) hide)
     )
@@
   (symbol (lib_id "MCU_Module:Arduino_UNO_R3") (at 252.73 52.07 0) (unit 1)
     (in_bom yes) (on_board yes) (fields_autoplaced)
-    (property "Reference" "A?" (id 0) (at 259.8294 24.13 0)
+    (property "Reference" "A1" (id 0) (at 259.8294 24.13 0)
       (effects (font (size 1.27 1.27)) (justify left))
     )
@@
       (effects (font (size 1.27 1.27)) (justify left))
     )
-    (property "Footprint" "Module:Arduino_UNO_R3" (id 2) (at 252.73 52.07 0)
+    (property "Footprint" "Module:Arduino_UNO_R3_WithMountingHoles" (id 2) (at 252.73 52.07 0)
       (effects (font (size 1.27 1.27) italic) hide)
     )
@@
   (symbol_instances
     (path "/7085cb2c-6e10-467e-a84c-9ccd4b76bee8"
-      (reference "#PWR04") (unit 1) (value "GND") (footprint "")
+      (reference "#PWR01") (unit 1) (value "GND") (footprint "")
     )
     (path "/9c6ca7ef-271b-4ee9-b9af-c9e07f71a58c"
-      (reference "#PWR07") (unit 1) (value "+3.3V") (footprint "")
+      (reference "#PWR02") (unit 1) (value "+3.3V") (footprint "")
     )
     (path "/4877b898-e2b7-449b-aa03-a14ce1f49e9b"
-      (reference "#PWR012") (unit 1) (value "GND") (footprint "")
+      (reference "#PWR03") (unit 1) (value "GND") (footprint "")
     )
     (path "/0ac43d98-b284-42fc-97e0-89a5e020d7c6"
-      (reference "#PWR013") (unit 1) (value "+3.3V") (footprint "")
+      (reference "#PWR04") (unit 1) (value "+3.3V") (footprint "")
     )
     (path "/d11df07d-6f34-43cd-a15d-c06df39a661d"
-      (reference "A?") (unit 1) (value "Arduino_UNO_R3") (footprint "Module:Arduino_UNO_R3")
+      (reference "A1") (unit 1) (value "Arduino_UNO_R3") (footprint "Module:Arduino_UNO_R3_WithMountingHoles")
     )
     (path "/80b61195-5427-4234-aff5-650722708293"

Commit message: Update PCB
Parts:
- added BZ1: Buzzer, Buzzer_Beeper:MagneticBuzzer_CUI_CMT-8504-100-SMT, symbol Device:Buzzer
- added C1: 0.1uF, Capacitor_SMD:C_0603_1608Metric_Pad1.08x0.95mm_HandSolder, symbol Device:C
- added D1, D2: D, Diode_SMD:D_SOD-123, symbol Device:D
- added J1: Conn_01x02, TerminalBlock_Phoenix:TerminalBlock_Phoenix_MKDS-1,5-2-5.08_1x02_P5.08mm_Horizontal, symbol Connector_Generic:Conn_01x02
- added J2: Temp, Connector_JST:JST_EH_S2B-EH_1x02_P2.50mm_Horizontal, symbol Connector_Generic:Conn_01x02
- added J4: SSR, Connector_JST:JST_EH_S2B-EH_1x02_P2.50mm_Horizontal, symbol Connector_Generic:Conn_01x02
- added J5: Fan, Connector_JST:JST_EH_S2B-EH_1x02_P2.50mm_Horizontal, symbol Connector_Generic:Conn_01x02
- added Q1, Q2, Q3: AO3400A, Package_TO_SOT_SMD:SOT-23_Handsoldering, symbol Transistor_FET:AO3400A
- added R1, R2, R3: R, Resistor_SMD:R_0603_1608Metric_Pad0.98x0.95mm_HandSolder, symbol Device:R
- A1: footprint Module:Arduino_UNO_R3_WithMountingHoles -> Module:Arduino_UNO_R3
- renumbered J1 to J3
Connections:
- net DO_TEMP is gone; now on net CS_MISO: IC1.7 (DO)
- net SCK_TEMP is gone; now on net CS_SCK: IC1.5 (SCK)
- net +3.3V: now also A1.4 (3V3), C1.1
- net CS_DISPLAY: now also A1.22 (D7)
- net CS_TEMP: now also A1.24 (D9)
- net CS_TOUCH: now also A1.18 (D3)
- net DC_DISPLAY: now also A1.20 (D5)
- net GND: now also A1.29 (GND), A1.6 (GND), A1.7 (GND), C1.2, J1.2 (Pin_2), Q1.2 (S), Q2.2 (S), Q3.2 (S), R1.2, R2.2, R3.2
- net IRQ_TOUCH: now also A1.17 (D2)
- net LED_DISPLAY: now also A1.19 (D4)
- net MISO: now also A1.27 (D12)
- net MOSI: now also A1.26 (D11)
- net RST_DISPLAY: now also A1.21 (D6)
- net SCK: now also A1.28 (D13)
- net heater_pins: now reaches A1.10 (A1)
- net heater_pins: now also Q1.1 (G), R1.1
- net FAN: now reaches A1.11 (A2)
- net FAN: now also Q2.1 (G), R2.1
- net CS_MISO: now reaches A1.23 (D8)
- net CS_SCK: now reaches A1.25 (D10)
- net +5V: now reaches A1.5 (+5V)
- net +5V: now also BZ1.1 (-), D1.1 (K), D2.1 (K), J4.1 (Pin_1), J5.1 (Pin_1)
- net V-IN: now reaches A1.8 (VIN)
- net V-IN: now also J1.1 (Pin_1)
- net BUZZER: now reaches A1.9 (A0)
- net BUZZER: now also Q3.1 (G), R3.1
- net T+: no longer names the net of IC1.3 (T+)
- net T+: now also J2.1 (Pin_1)
- net T-: no longer names the net of IC1.2 (T-)
- net T-: now also J2.2 (Pin_2)
- new net: J4.2 (Pin_2), Q1.3 (D)
- new net: BZ1.2 (+), D2.2 (A), Q3.3 (D)
- new net: D1.2 (A), J5.2 (Pin_2), Q2.3 (D)
Other:
- moved on the sheet: A1, IC1, J3
